Commit message: moveit test finish

File: src/manipulator_moveit/config/manipulator.ros2_control.xacro (robot description, xacro)
@@ -2,5 +2,5 @@
 <robot xmlns:xacro="http://www.ros.org/wiki/xacro">
     <xacro:macro name="manipulator_ros2_control" params="name initial_positions_file">
-        <xacro:property name="initial_positions" value="${load_yaml(initial_positions_file)['initial_positions']}"/>
+        <xacro:property name="initial_positions" value="${xacro.load_yaml(initial_positions_file)['initial_positions']}"/>
         <ros2_control name="${name}" type="system">
             <hardware>

File: src/manipulator_moveit/config/manipulator.urdf.xacro (robot description, xacro)
@@ -1,9 +1,9 @@
 <?xml version="1.0"?>
 <robot xmlns:xacro="http://www.ros.org/wiki/xacro" name="open_manipulator_x">
-    <xacro:arg name="initial_positions_file" default="initial_positions.yaml" />
+    <xacro:arg name="initial_positions_file" default="$(find manipulator_moveit)/config/initial_positions.yaml" />
     <!-- Import open_manipulator_x urdf file -->
-    <xacro:include filename="$(find manipulator_description)/description/capstone_manipulator.urdf.xacro" />
+    <xacro:include filename="$(find manipulator)/description/capstone_manipulator.urdf.xacro" />
     <!-- Import control_xacro -->
     <xacro:include filename="manipulator.ros2_control.xacro" />
-    <xacro:open_manipulator_x_ros2_control name="FakeSystem" initial_positions_file="$(arg initial_positions_file)"/>
+    <xacro:manipulator_ros2_control name="FakeSystem" initial_positions_file="$(arg initial_positions_file)"/>
 </robot>
