Commit message: sym error solution

File: src/manipulator/description/capstone_manipulator.urdf.xacro (robot description, xacro)
@@ -1 +1,211 @@
-/home/moonshot/open_manipulator/src/open_manipulator_x_description/urdf/capstone_manipulator.urdf.xacro
+<?xml version="1.0" ?>
+<!-- =================================================================================== -->
+<!-- |    This document was autogenerated by xacro from capstone_manipulator.urdf.xacro | -->
+<!-- |    EDITING THIS FILE BY HAND IS NOT RECOMMENDED                                 | -->
+<!-- =================================================================================== -->
+<robot name="manipulator">
+  <!-- Optional materials for RViz -->
+  <material name="grey">
+    <color rgba="0.2 0.2 0.2 1.0"/>
+  </material>
+  <material name="dark_grey">
+    <color rgba="0.05 0.05 0.05 1.0"/>
+  </material>
+  <material name="red">
+    <color rgba="0.6 0.1 0.1 1.0"/>
+  </material>
+  <!-- =========================
+       link1 (base block on robot, bottom at z=0)
+       size: 0.05 x 0.05 x 0.05
+       ========================= -->
+  <link name="link1">
+    <visual>
+      <origin rpy="0 0 0" xyz="0 0 0.025"/>
+      <geometry>
+        <box size="0.05 0.05 0.05"/>
+      </geometry>
+      <material name="dark_grey"/>
+    </visual>
+    <collision>
+      <origin rpy="0 0 0" xyz="0 0 0.025"/>
+      <geometry>
+        <box size="0.05 0.05 0.05"/>
+      </geometry>
+    </collision>
+    <inertial>
+      <origin rpy="0 0 0" xyz="0 0 0.025"/>
+      <mass value="1.0"/>
+      <inertia ixx="0.0004166667" ixy="0" ixz="0" iyy="0.0004166667" iyz="0" izz="0.0004166667"/>
+    </inertial>
+  </link>
+  <!-- joint1: base yaw (Z) -->
+  <joint name="joint1" type="revolute">
+    <parent link="link1"/>
+    <child link="link2"/>
+    <origin rpy="0 0 0" xyz="0 0 0.05"/>
+    <axis xyz="0 0 1"/>
+    <limit effort="0.1" lower="-3.14159265359" upper="3.14159265359" velocity="4.8"/>
+  </joint>
+  <!-- =========================
+       link2 (vertical riser)
+       length: 0.12m, cross-section: 0.05 x 0.05
+       ========================= -->
+  <link name="link2">
+    <visual>
+      <origin rpy="0 0 0" xyz="0 0 0.06"/>
+      <geometry>
+        <box size="0.05 0.05 0.12"/>
+      </geometry>
+      <material name="grey"/>
+    </visual>
+    <collision>
+      <origin rpy="0 0 0" xyz="0 0 0.06"/>
+      <geometry>
+        <box size="0.05 0.05 0.12"/>
+      </geometry>
+    </collision>
+    <inertial>
+      <origin rpy="0 0 0" xyz="0 0 0.06"/>
+      <mass value="0.8"/>
+      <inertia ixx="0.0019866667" ixy="0" ixz="0" iyy="0.0019866667" iyz="0" izz="0.0003333333"/>
+    </inertial>
+  </link>
+  <!-- joint2: shoulder pitch (Y) at top of link2 -->
+  <joint name="joint2" type="revolute">
+    <parent link="link2"/>
+    <child link="link3"/>
+    <origin rpy="0 0 0" xyz="0 0 0.12"/>
+    <axis xyz="0 1 0"/>
+    <limit effort="0.1" lower="-3.14159265359" upper="0.785398" velocity="4.8"/>
+  </joint>
+  <!-- =========================
+       link3 (upper arm)
+       length: 0.30m along +X, cross-section: 0.05 x 0.05
+       ========================= -->
+  <link name="link3">
+    <visual>
+      <origin rpy="0 0 0" xyz="0.15 0 0"/>
+      <geometry>
+        <box size="0.30 0.05 0.05"/>
+      </geometry>
+      <material name="grey"/>
+    </visual>
+    <collision>
+      <origin rpy="0 0 0" xyz="0.15 0 0"/>
+      <geometry>
+        <box size="0.30 0.05 0.05"/>
+      </geometry>
+    </collision>
+    <inertial>
+      <origin rpy="0 0 0" xyz="0.15 0 0"/>
+      <mass value="0.6"/>
+      <inertia ixx="0.0002500000" ixy="0" ixz="0" iyy="0.0046250000" iyz="0" izz="0.0046250000"/>
+    </inertial>
+  </link>
+  <!-- joint3: elbow pitch (Y) at end of link3 -->
+  <joint name="joint3" type="revolute">
+    <parent link="link3"/>
+    <child link="link4"/>
+    <origin rpy="0 0 0" xyz="0.30 0 0"/>
+    <axis xyz="0 1 0"/>
+    <limit effort="0.1" lower="0" upper="2.7" velocity="4.8"/>
+  </joint>
+  <!-- =========================
+       link4 (forearm)
+       length: 0.30m along +X
+       ========================= -->
+  <link name="link4">
+    <visual>
+      <origin rpy="0 0 0" xyz="0.15 0 0"/>
+      <geometry>
+        <box size="0.30 0.05 0.05"/>
+      </geometry>
+      <material name="grey"/>
+    </visual>
+    <collision>
+      <origin rpy="0 0 0" xyz="0.15 0 0"/>
+      <geometry>
+        <box size="0.30 0.05 0.05"/>
+      </geometry>
+    </collision>
+    <inertial>
+      <origin rpy="0 0 0" xyz="0.15 0 0"/>
+      <mass value="0.5"/>
+      <inertia ixx="0.0002083333" ixy="0" ixz="0" iyy="0.0038541667" iyz="0" izz="0.0038541667"/>
+    </inertial>
+  </link>
+  <!-- joint4: wrist pitch (Y) at end of link4 -->
+  <joint name="joint4" type="revolute">
+    <parent link="link4"/>
+    <child link="link5"/>
+    <origin rpy="0 0 0" xyz="0.30 0 0"/>
+    <axis xyz="0 1 0"/>
+    <limit effort="0.1" lower="-1.5" upper="1.5" velocity="4.8"/>
+  </joint>
+  <link name="link5">
+    <visual>
+      <origin rpy="0 0 0" xyz="0.05 0 0"/>
+      <geometry>
+        <box size="0.10 0.03 0.03"/>
+      </geometry>
+      <material name="red"/>
+    </visual>
+    <collision>
+      <origin rpy="0 0 0" xyz="0.05 0 0"/>
+      <geometry>
+        <box size="0.10 0.03 0.03"/>
+      </geometry>
+    </collision>
+    <inertial>
+      <origin rpy="0 0 0" xyz="0.05 0 0"/>
+      <mass value="0.2"/>
+      <inertia ixx="0.0000300000" ixy="0" ixz="0" iyy="0.0001766667" iyz="0" izz="0.0001766667"/>
+    </inertial>
+  </link>
+  <link name="ee_link">
+    <visual>
+      <origin rpy="0 0 0" xyz="0 0 0"/>
+      <geometry>
+        <box size="0.01 0.01 0.01"/>
+      </geometry>
+      <material name="dark_grey"/>
+    </visual>
+    <collision>
+      <origin rpy="0 0 0" xyz="0 0 0"/>
+      <geometry>
+        <box size="0.01 0.01 0.01"/>
+      </geometry>
+    </collision>
+    <inertial>
+      <origin rpy="0 0 0" xyz="0 0 0"/>
+      <mass value="0.05"/>
+      <inertia ixx="0.0000008333" ixy="0" ixz="0" iyy="0.0000008333" iyz="0" izz="0.0000008333"/>
+    </inertial>
+  </link>
+  <joint name="ee_fixed_joint" type="fixed">
+    <parent link="link5"/>
+    <child link="ee_link"/>
+    <origin rpy="0 0 0" xyz="0.10 0 0"/>
+  </joint>
+  <!-- RealSense Camera Link -->
+  <link name="camera_link">
+    <visual>
+      <origin rpy="0 0 0" xyz="0 0 0"/>
+      <geometry>
+        <box size="0.025 0.09 0.025"/>
+      </geometry>
+      <material name="dark_grey"/>
+    </visual>
+    <inertial>
+      <origin rpy="0 0 0" xyz="0 0 0"/>
+      <mass value="0.1"/>
+      <inertia ixx="0.0000735417" ixy="0" ixz="0" iyy="0.0000020833" iyz="0" izz="0.0000735417"/>
+    </inertial>
+  </link>
+  <!-- Joint connecting last link and camera_link  -->
+  <joint name="camera_joint" type="fixed">
+    <parent link="link5"/>
+    <child link="camera_link"/>
+    <origin rpy="0 0 0" xyz="0.04 0.0 0.027"/>
+  </joint>
+</robot>
